Commit message: launch file edit

File: description/testbot.xacro (robot description, xacro)
@@ -182,4 +182,31 @@
     <origin xyz="0 0 0.01"/>
   </joint>
+    <!--Control ad gazebo control interface-->
+    <ros2_control name="IgnitionSystem" type="system">
+    <hardware>
+      <plugin>ign_ros2_control/IgnitionSystem</plugin>
+    </hardware>
+    <joint name="base_right_wheel">
+      <command_interface name="velocity">
+        <param name="min">-1</param>
+        <param name="max">1</param>
+      </command_interface>
+      <state_interface name="position"/>
+      <state_interface name="velocity"/>
+    </joint>
+    <joint name="base_left_wheel">
+      <command_interface name="velocity">
+        <param name="min">-1</param>
+        <param name="max">1</param>
+      </command_interface>
+      <state_interface name="position"/>
+      <state_interface name="velocity"/>
+    </joint>
+  </ros2_control>
+  <gazebo>
+    <plugin filename="ign_ros2_control-system" name="ign_ros2_control::IgnitionROS2ControlPlugin">
+      <parameters>$(find testbot)/config/diff_drive_controller_velocity.yaml</parameters>
+    </plugin>
+  </gazebo>
   <!--Camera properties-->
 </robot>

Commit message: odom fixing

File: description/testbot.xacro (robot description, xacro)
@@ -1,4 +1,4 @@
 <?xml version="1.0"?>
-<robot xmlns:xacro="http://www.ros.org/wiki/xacro" >
+<robot xmlns:xacro="http://www.ros.org/wiki/xacro" name="roboct" >
 <!---materials definitions-->
 <material name="green">
@@ -33,5 +33,5 @@
             <box size="0.6 0.4 0.2"/>
         </geometry>
-        <origin xyz="0.0 0.0 0.1" rpy="0.0 0.0 0.0"/>
+        <origin xyz="0.0 0.0 0.05" rpy="0.0 0.0 0.0"/>
         <material name="green"/>
     </visual>
@@ -40,12 +40,12 @@
             <box size="0.6 0.4 0.2"/>
         </geometry>
-        <origin xyz="0.0 0.0 0.1" rpy="0.0 0.0 0.0"/>
+        <origin xyz="0.0 0.0 0.05" rpy="0.0 0.0 0.0"/>
     </collision>
     <xacro:box_inertia m="1.0" w="0.4" d="0.6" h="0.2"/>
 </link>
 <joint name="base_link_footprint_joint" type="fixed">
-    <origin xyz="0.0 0.0 0.1" rpy="0.0 0.0 0.0"/>
-    <parent link="base_footprint"/>
-    <child link="base_link"/>
+    <origin xyz="0.0 0.0 -0.15" rpy="0.0 0.0 0.0"/>
+    <parent link="base_link"/>
+    <child link="base_footprint"/>
 </joint>
 <!--Lidar properties-->
@@ -98,10 +98,9 @@
 </link>
 <joint name="base_left_wheel" type="continuous">
-    <origin xyz="-0.15 0.225 0.0" rpy="0.0 0.0 0.0"/>
+    <origin xyz="-0.15 0.233 0.0" rpy="0.0 0.0 0.0"/>
     <parent link="base_link"/>
     <child link="left_wheel"/>
     <axis xyz="0.0 1.0 0.0"/>
-    <limit lower="0.0" upper="0.0" effort="0.0" velocity="1000.0"/>
-    <dynamics damping="1.0" friction="1.0"/>
+    <dynamics damping="0.2"/>
 </joint>
 <!--Right Wheel properties-->
@@ -127,10 +126,9 @@
 </link>
 <joint name="base_right_wheel" type="continuous">
-    <origin xyz="-0.15 -0.225 0.0" rpy="0.0 0.0 0.0"/>
+    <origin xyz="-0.15 -0.233 0.0" rpy="0.0 0.0 0.0"/>
     <parent link="base_link"/>
     <child link="right_wheel"/>
     <axis xyz="0.0 1.0 0.0"/>
-    <limit lower="0.0" upper="0.0" effort="0.0" velocity="1000.0"/>
-    <dynamics damping="1.0" friction="1.0"/>
+    <dynamics damping="0.2"/>
 </joint>
 <!--Caster Wheel properties-->
