Commit message: sdf edit

File: description/robot.urdf.xacro (robot description, xacro)
@@ -1,160 +1,4 @@
 <?xml version="1.0"?>
 <robot xmlns:xacro="http://www.ros.org/wiki/xacro"  name="roboct">
-<material name="green">
-    <color rgba="0.0 0.7 0.0 1.0"/>
-</material>
-<material name="blue">
-<color rgba="0.0 0.0 1.0 1.0"/>
-</material>
-<material name="red">
-    <color rgba="1.0 0.0 0.0 1.0"/>
-</material>
-<material name="white">
-    <color rgba="1.0 1.0 1.0 1.0"/>
-</material>
-<material name="black">
-    <color rgba="0.0 0.0 0.0 1.0"/>
-</material>
-<!--- All Robots links-->
-<!--Base_link properties-->
-<link name="base_footprint"/>
-<link name="base_link">
-    <visual>
-        <geometry>
-            <box size="0.6 0.4 0.2"/>
-        </geometry>
-        <origin xyz="0.0 0.0 0.1" rpy="0.0 0.0 0.0"/>
-        <material name="green"/>
-    </visual>
-    <collision>
-        <geometry>
-            <box size="0.6 0.4 0.2"/>
-        </geometry>
-        <origin xyz="0.0 0.0 0.1" rpy="0.0 0.0 0.0"/>
-    </collision>
-    <inertial>
-        <mass value="1.0"/>
-        <origin xyz="0 0 0.1"/> <!-- Assuming the center of mass is at the origin -->
-        <inertia ixx="0.0167" ixy="0.0" ixz="0.0" iyy="0.0333" iyz="0.0" izz="0.0433"/>
-    </inertial>
-</link>
-<!--Lidar properties-->
-<link name = "lidar">
-    <visual>
-            <geometry>
-                <cylinder radius="0.1" length="0.05"/>
-            </geometry>
-            <origin xyz="0.0 0.0 0.0" rpy="0.0 0.0 0.0"/>
-            <material name="black"/>
-    </visual>
-    <collision>
-        <geometry>
-            <cylinder radius="0.1" length="0.05"/>
-        </geometry>
-    </collision>
-    <inertial>
-            <mass value="1.0"/>
-            <origin xyz="0 0 0"/>
-            <inertia ixx="0.001458" iyy="0.001458" izz="0.00125" ixy="0.0" ixz="0.0" iyz="0.0"/>
-    </inertial>
-</link>
-<!--Left Wheel properties-->
-<link name = "left_wheel">
-    <visual>
-            <geometry>
-                <cylinder radius="0.1" length="0.05"/>
-            </geometry>
-            <origin xyz="0.0 0.0 0.0" rpy="1.57 0.0 0.0"/>
-            <material name="blue"/>
-    </visual>
-    <collision>
-        <geometry>
-            <cylinder radius="0.1" length="0.05"/>
-        </geometry>
-        <origin xyz="0.0 0.0 0.0" rpy="1.57 0.0 0.0"/>
-    </collision>
-    <inertial>
-            <mass value="1.0"/>
-            <origin xyz="0 0 0"/>
-            <inertia ixx="0.001458" iyy="0.001458" izz="0.00125" ixy="0.0" ixz="0.0" iyz="0.0"/>
-    </inertial>
-</link>
-<!--Right Wheel properties-->
-<link name = "right_wheel">
-    <visual>
-            <geometry>
-                <cylinder radius="0.1" length="0.05"/>
-            </geometry>
-            <origin xyz="0.0 0.0 0.0" rpy="1.570 0.0 0.0"/>
-            <material name="blue"/>
-    </visual>
-    <collision>
-        <geometry>
-            <cylinder radius="0.1" length="0.05"/>
-        </geometry>
-        <origin xyz="0.0 0.0 0.0" rpy="1.57 0.0 0.0"/>
-    </collision>
-    <inertial>
-        <mass value="1.0"/>
-        <origin xyz="0 0 0"/>
-        <inertia ixx="0.001458" iyy="0.001458" izz="0.00125" ixy="0.0" ixz="0.0" iyz="0.0"/>
-    </inertial>
-</link>
-<!--Caster Wheel properties-->
-<link name = "caster_wheel">
-<visual>
-        <geometry>
-            <sphere radius="0.05"/>
-        </geometry>
-        <origin xyz="0.0 0.0 0.0" rpy="0.0 0.0 0.0"/>
-        <material name="white"/>
-</visual>
-<collision>
-        <geometry>
-            <sphere radius="0.05"/>
-        </geometry>
-</collision>
-<inertial>
-    <origin xyz="0 0 0" rpy="0 0 0"/> <!-- Assume the center of mass is at the origin -->
-    <mass value="1.0"/>
-    <inertia ixx="0.001" ixy="0.0" ixz="0.0" iyy="0.001" iyz="0.0" izz="0.001"/>
-  </inertial>
-</link>
-<!--- All joints for links-->
-<joint name="base_lidar" type="fixed">
-    <origin xyz="0.0 0.0 0.225" rpy="0.0 0.0 0.0"/>
-    <parent link="base_link"/>
-    <child link="lidar"/>
-    <axis xyz="0.0 0.0 0.0"/>
-    <limit lower="0.0" upper="0.0" effort="0.0" velocity="0.0"/>
-</joint>
-<joint name="base_left_wheel" type="continuous">
-    <origin xyz="-0.15 0.225 0.0" rpy="0.0 0.0 0.0"/>
-    <parent link="base_link"/>
-    <child link="left_wheel"/>
-    <axis xyz="0.0 1.0 0.0"/>
-    <limit lower="0.0" upper="0.0" effort="0.0" velocity="1000.0"/>
-    <dynamics damping="1.0" friction="1.0"/>
-</joint>
-<joint name="base_right_wheel" type="continuous">
-    <origin xyz="-0.15 -0.225 0.0" rpy="0.0 0.0 0.0"/>
-    <parent link="base_link"/>
-    <child link="right_wheel"/>
-    <axis xyz="0.0 1.0 0.0"/>
-    <limit lower="0.0" upper="0.0" effort="0.0" velocity="1000.0"/>
-    <dynamics damping="1.0" friction="1.0"/>
-</joint>
-<joint name="base_caster" type="fixed">
-    <origin xyz="0.2 0.0 -0.04" rpy="0.0 0.0 0.0"/>
-    <parent link="base_link"/>
-    <child link="caster_wheel"/>
-    <axis xyz="0.0 0.0 0.0"/>
-    <limit lower="0.0" upper="0.0" effort="0.0" velocity="0.0"/>
-    <dynamics damping="1.0" friction="1.0"/>
-</joint>
-<joint name="joint_name" type="fixed">
-    <origin xyz="0.0 0.0 0.1" rpy="0.0 0.0 0.0"/>
-    <parent link="base_footprint"/>
-    <child link="base_link"/>
-</joint>
+    <xacro:include filename="testbot.xacro"/>
 </robot>

Commit message: added sim vid

File: description/robot.urdf.xacro (robot description, xacro)
@@ -1,4 +1,204 @@
 <?xml version="1.0"?>
-<robot xmlns:xacro="http://www.ros.org/wiki/xacro"  name="roboct">
-    <xacro:include filename="testbot.xacro"/>
+<robot xmlns:xacro="http://www.ros.org/wiki/xacro" name="roboct" >
+<!---materials definitions-->
+<material name="green">
+    <color rgba="0.0 0.7 0.0 1.0"/>
+</material>
+<material name="blue">
+<color rgba="0.0 0.0 1.0 1.0"/>
+</material>
+<material name="red">
+    <color rgba="1.0 0.0 0.0 1.0"/>
+</material>
+<material name="white">
+    <color rgba="1.0 1.0 1.0 1.0"/>
+</material>
+<material name="black">
+    <color rgba="0.0 0.0 0.0 1.0"/>
+</material>
+<!-- Define some commonly used intertial properties  -->
+  <xacro:macro name="box_inertia" params="m w h d">
+    <inertial>
+      <origin xyz="0 0 0" rpy="${pi/2} 0 ${pi/2}"/>
+      <mass value="${m}"/>
+      <inertia ixx="${(m/12) * (h*h + d*d)}" ixy="0.0" ixz="0.0" iyy="${(m/12) * (w*w + d*d)}" iyz="0.0" izz="${(m/12) * (w*w + h*h)}"/>
+    </inertial>
+  </xacro:macro>
+<!--- All Robots links with their full properties-->
+<!--Base_link properties-->
+<link name="base_footprint"/>
+<link name="base_link">
+    <visual>
+        <geometry>
+            <box size="0.6 0.4 0.2"/>
+        </geometry>
+        <origin xyz="0.0 0.0 0.05" rpy="0.0 0.0 0.0"/>
+        <material name="green"/>
+    </visual>
+    <collision>
+        <geometry>
+            <box size="0.6 0.4 0.2"/>
+        </geometry>
+        <origin xyz="0.0 0.0 0.05" rpy="0.0 0.0 0.0"/>
+    </collision>
+    <xacro:box_inertia m="1.0" w="0.4" d="0.6" h="0.2"/>
+</link>
+<joint name="base_link_footprint_joint" type="fixed">
+    <origin xyz="0.0 0.0 -0.15" rpy="0.0 0.0 0.0"/>
+    <parent link="base_link"/>
+    <child link="base_footprint"/>
+</joint>
+<!--Lidar properties-->
+<link name = "lidar">
+    <visual>
+            <geometry>
+                <cylinder radius="0.1" length="0.05"/>
+            </geometry>
+            <origin xyz="0.0 0.0 0.0" rpy="0.0 0.0 0.0"/>
+            <material name="black"/>
+    </visual>
+    <collision>
+        <geometry>
+            <cylinder radius="0.1" length="0.05"/>
+        </geometry>
+    </collision>
+    <inertial>
+            <mass value="1.0"/>
+            <origin xyz="0 0 0"/>
+            <inertia ixx="0.001458" iyy="0.001458" izz="0.00125" ixy="0.0" ixz="0.0" iyz="0.0"/>
+    </inertial>
+</link>
+<joint name="base_lidar" type="fixed">
+    <origin xyz="0.0 0.0 0.225" rpy="0.0 0.0 0.0"/>
+    <parent link="base_link"/>
+    <child link="lidar"/>
+    <axis xyz="0.0 0.0 0.0"/>
+    <limit lower="0.0" upper="0.0" effort="0.0" velocity="0.0"/>
+</joint>
+<!--Left Wheel properties-->
+<link name = "left_wheel">
+    <visual>
+            <geometry>
+                <cylinder radius="0.1" length="0.05"/>
+            </geometry>
+            <origin xyz="0.0 0.0 0.0" rpy="1.57 0.0 0.0"/>
+            <material name="blue"/>
+    </visual>
+    <collision>
+        <geometry>
+            <cylinder radius="0.1" length="0.05"/>
+        </geometry>
+        <origin xyz="0.0 0.0 0.0" rpy="1.57 0.0 0.0"/>
+    </collision>
+    <inertial>
+            <mass value="1.0"/>
+            <origin xyz="0 0 0"/>
+            <inertia ixx="0.001458" iyy="0.001458" izz="0.00125" ixy="0.0" ixz="0.0" iyz="0.0"/>
+    </inertial>
+</link>
+<joint name="base_left_wheel" type="continuous">
+    <origin xyz="-0.15 0.233 0.0" rpy="0.0 0.0 0.0"/>
+    <parent link="base_link"/>
+    <child link="left_wheel"/>
+    <axis xyz="0.0 1.0 0.0"/>
+    <dynamics damping="0.2"/>
+</joint>
+<!--Right Wheel properties-->
+<link name = "right_wheel">
+    <visual>
+            <geometry>
+                <cylinder radius="0.1" length="0.05"/>
+            </geometry>
+            <origin xyz="0.0 0.0 0.0" rpy="1.570 0.0 0.0"/>
+            <material name="blue"/>
+    </visual>
+    <collision>
+        <geometry>
+            <cylinder radius="0.1" length="0.05"/>
+        </geometryixx="0.001458" iyy="0.001458" izz="0.00125" ixy="0.0" ixz="0.0" iyz="0.0"/>
+    </inertial>
+</link>
+<joint name="base_right_wheel" type="continuous">
+    <origin xyz="-0.15 -0.233 0.0" rpy="0.0 0.0 0.0"/>
+    <parent link="base_link"/>
+    <child link="right_wheel"/>
+    <axis xyz="0.0 1.0 0.0"/>
+    <dynamics damping="0.2"/>
+</joint>
+<!--Caster Wheel properties-->
+<link name = "caster_wheel">
+<visual>
+        <geometry>
+            <sphere radius="0.05"/>
+        </geometry>
+        <origin xyz="0.0 0.0 0.0" rpy="0.0 0.0 0.0"/>
+        <material name="white"/>
+</visual>
+<collision>
+        <geometry>
+            <sphere radius="0.05"/>
+        </geometry>
+</collision>
+<inertial>
+    <origin xyz="0 0 0" rpy="0 0 0"/> <!-- Assume the center of mass is at the origin -->
+    <mass value="1.0"/>
+    <inertia ixx="0.001" ixy="0.0" ixz="0.0" iyy="0.001" iyz="0.0" izz="0.001"/>
+  </inertial>
+</link>
+<joint name="base_caster" type="fixed">
+    <origin xyz="0.2 0.0 -0.04" rpy="0.0 0.0 0.0"/>
+    <parent link="base_link"/>
+    <child link="caster_wheel"/>
+    <axis xyz="0.0 0.0 0.0"/>
+    <limit lower="0.0" upper="0.0" effort="0.0" velocity="0.0"/>
+    <dynamics damping="1.0" friction="1.0"/>
+</joint>
+<!---IMU properties-->
+<link name="imu_link">
+    <visual>
+      <geometry>
+        <box size="0.1 0.1 0.1"/>
+      </geometry>
+      <material name="red"/>
+    </visual>
+    <collision>
+      <geometry>
+        <box size="0.1 0.1 0.1"/>
+      </geometry>
+    </collision>
+    <xacro:box_inertia m="0.001" w="0.1" d="0.1" h="0.1"/>
+  </link>
+   <joint name="imu_joint" type="fixed">
+    <parent link="base_link"/>
+    <child link="imu_link"/>
+    <origin xyz="0 0 0.01"/>
+  </joint>
+    <!--Control ad gazebo control interface-->
+    <ros2_control name="IgnitionSystem" type="system">
+    <hardware>
+      <plugin>ign_ros2_control/IgnitionSystem</plugin>
+    </hardware>
+    <joint name="base_right_wheel">
+      <command_interface name="velocity">
+        <param name="min">-1</param>
+        <param name="max">1</param>
+      </command_interface>
+      <state_interface name="position"/>
+      <state_interface name="velocity"/>
+    </joint>
+    <joint name="base_left_wheel">
+      <command_interface name="velocity">
+        <param name="min">-1</param>
+        <param name="max">1</param>
+      </command_interface>
+      <state_interface name="position"/>
+      <state_interface name="velocity"/>
+    </joint>
+  </ros2_control>
+  <gazebo>
+    <plugin filename="ign_ros2_control-system" name="ign_ros2_control::IgnitionROS2ControlPlugin">
+      <parameters>$(find testbot)/config/diff_drive_controller_velocity.yaml</parameters>
+    </plugin>
+  </gazebo>
+  <!--Camera properties-->
 </robot>

File: description/testbot.xacro (robot description, xacro)
@@ -120,7 +120,7 @@
     </collision>
     <inertial>
-        <mass value="1.0"/>
-        <origin xyz="0 0 0"/>
-        <inertia ixx="0.001458" iyy="0.001458" izz="0.00125" ixy="0.0" ixz="0.0" iyz="0.0"/>
+            <mass value="1.0"/>
+            <origin xyz="0 0 0"/>
+            <inertia ixx="0.001458" iyy="0.001458" izz="0.00125" ixy="0.0" ixz="0.0" iyz="0.0"/>
     </inertial>
 </link>
