Commit message: created 4wheel

File: description/4w_testbot.xacro (robot description, xacro)
@@ -53,5 +53,5 @@
     <visual>
             <geometry>
-                <cylinder radius="0.1" length="0.05"/>
+                <cylinder radius="0.0808" length="0.055"/>
             </geometry>
             <origin xyz="0.0 0.0 0.0" rpy="0.0 0.0 0.0"/>
@@ -60,5 +60,5 @@
     <collision>
         <geometry>
-            <cylinder radius="0.1" length="0.05"/>
+            <cylinder radius="0.0808" length="0.055"/>
         </geometry>
     </collision>
@@ -70,5 +70,5 @@
 </link>
 <joint name="base_lidar" type="fixed">
-    <origin xyz="0.0 0.0 0.225" rpy="0.0 0.0 0.0"/>
+    <origin xyz="0.0 0.0 0.2" rpy="0.0 0.0 0.0"/>
     <parent link="base_link"/>
     <child link="lidar"/>
@@ -76,11 +76,12 @@
     <limit lower="0.0" upper="0.0" effort="0.0" velocity="0.0"/>
 </joint>
-<!--Left Wheel properties-->
-<link name = "left_wheel">
+<!--Wheel properties-->
+<xacro:macro name="wheel" params="name xyz rpy jrpy">
+<link name = "${name}">
     <visual>
             <geometry>
                 <cylinder radius="0.1" length="0.05"/>
             </geometry>
-            <origin xyz="0.0 0.0 0.0" rpy="1.57 0.0 0.0"/>
+            <origin xyz="0.0 0.0 0.0" rpy="${rpy}"/>
             <material name="blue"/>
     </visual>
@@ -89,5 +90,5 @@
             <cylinder radius="0.1" length="0.05"/>
         </geometry>
-        <origin xyz="0.0 0.0 0.0" rpy="1.57 0.0 0.0"/>
+        <origin xyz="0.0 0.0 0.0" rpy="${rpy}"/>
     </collision>
     <inertial>
@@ -97,67 +98,17 @@
     </inertial>
 </link>
-<joint name="base_left_wheel" type="continuous">
-    <origin xyz="-0.15 0.233 0.0" rpy="0.0 0.0 0.0"/>
+<joint name="${name}_joint" type="continuous">
+    <origin xyz="${xyz}" rpy="0 0 0"/>
     <parent link="base_link"/>
-    <child link="left_wheel"/>
+    <child link="${name}"/>
     <axis xyz="0.0 1.0 0.0"/>
     <dynamics damping="0.2"/>
 </joint>
-<!--Right Wheel properties-->
-<link name = "right_wheel">
-    <visual>
-            <geometry>
-                <cylinder radius="0.1" length="0.05"/>
-            </geometry>
-            <origin xyz="0.0 0.0 0.0" rpy="1.570 0.0 0.0"/>
-            <material name="blue"/>
-    </visual>
-    <collision>
-        <geometry>
-            <cylinder radius="0.1" length="0.05"/>
-        </geometry>
-        <origin xyz="0.0 0.0 0.0" rpy="1.57 0.0 0.0"/>
-    </collision>
-    <inertial>
-            <mass value="1.0"/>
-            <origin xyz="0 0 0"/>
-            <inertia ixx="0.001458" iyy="0.001458" izz="0.00125" ixy="0.0" ixz="0.0" iyz="0.0"/>
-    </inertial>
-</link>
-<joint name="base_right_wheel" type="continuous">
-    <origin xyz="-0.15 -0.233 0.0" rpy="0.0 0.0 0.0"/>
-    <parent link="base_link"/>
-    <child link="right_wheel"/>
-    <axis xyz="0.0 1.0 0.0"/>
-    <dynamics damping="0.2"/>
-</joint>
-<!--Caster Wheel properties-->
-<link name = "caster_wheel">
-<visual>
-        <geometry>
-            <sphere radius="0.05"/>
-        </geometry>
-        <origin xyz="0.0 0.0 0.0" rpy="0.0 0.0 0.0"/>
-        <material name="white"/>
-</visual>
-<collision>
-        <geometry>
-            <sphere radius="0.05"/>
-        </geometry>
-</collision>
-<inertial>
-    <origin xyz="0 0 0" rpy="0 0 0"/> <!-- Assume the center of mass is at the origin -->
-    <mass value="1.0"/>
-    <inertia ixx="0.001" ixy="0.0" ixz="0.0" iyy="0.001" iyz="0.0" izz="0.001"/>
-  </inertial>
-</link>
-<joint name="base_caster" type="fixed">
-    <origin xyz="0.2 0.0 -0.04" rpy="0.0 0.0 0.0"/>
-    <parent link="base_link"/>
-    <child link="caster_wheel"/>
-    <axis xyz="0.0 0.0 0.0"/>
-    <limit lower="0.0" upper="0.0" effort="0.0" velocity="0.0"/>
-    <dynamics damping="1.0" friction="1.0"/>
-</joint>
+</xacro:macro>
+<!--definition of all four wheels-->
+<xacro:wheel name="rr_wheel" xyz="-0.18 -0.233 0.0" rpy="1.57 0 0" jrpy="3.142 0.0 0.0"/> <!--Rear right wheel-->
+<xacro:wheel name="fr_wheel" xyz="0.18 -0.233 0.0" rpy="1.57 0 0" jrpy="3.142 0.0 0.0"/><!--front right wheel-->
+<xacro:wheel name="fl_wheel" xyz="0.18 0.233 0.0" rpy="1.57 0 0" jrpy="0.0 0.0 0.0"/><!--front left wheel-->
+<xacro:wheel name="rl_wheel" xyz="-0.18 0.233 0.0" rpy="1.57 0 0" jrpy="0.0 0.0 0.0"/><!--rear leftwheel-->
 <!---IMU properties-->
 <link name="imu_link">
@@ -185,5 +136,5 @@
       <plugin>ign_ros2_control/IgnitionSystem</plugin>
     </hardware>
-    <joint name="base_right_wheel">
+    <joint name="fr_wheel_joint">
       <command_interface name="velocity">
         <param name="min">-1</param>
@@ -193,5 +144,21 @@
       <state_interface name="velocity"/>
     </joint>
-    <joint name="base_left_wheel">
+    <joint name="rr_wheel_joint">
+      <command_interface name="velocity">
+        <param name="min">-1</param>
+        <param name="max">1</param>
+      </command_interface>
+      <state_interface name="position"/>
+      <state_interface name="velocity"/>
+    </joint>
+    <joint name="fl_wheel_joint">
+      <command_interface name="velocity">
+        <param name="min">-1</param>
+        <param name="max">1</param>
+      </command_interface>
+      <state_interface name="position"/>
+      <state_interface name="velocity"/>
+    </joint>
+    <joint name="rl_wheel_joint">
       <command_interface name="velocity">
         <param name="min">-1</param>
@@ -204,5 +171,5 @@
   <gazebo>
     <plugin filename="ign_ros2_control-system" name="ign_ros2_control::IgnitionROS2ControlPlugin">
-      <parameters>$(find testbot)/config/diff_drive_controller_velocity.yaml</parameters>
+      <parameters>$(find testbot)/config/4w_diff_drive_controller_velocity.yaml</parameters>
     </plugin>
   </gazebo>

Commit message: CMakelist edit

File: description/4w_testbot.xacro (robot description, xacro)
@@ -50,10 +50,9 @@
 </joint>
 <!--Lidar properties-->
-<link name = "lidar">
+ <link name = "lidar_link">
     <visual>
             <geometry>
                 <cylinder radius="0.0808" length="0.055"/>
             </geometry>
-            <origin xyz="0.0 0.0 0.0" rpy="0.0 0.0 0.0"/>
             <material name="black"/>
     </visual>
@@ -65,5 +64,4 @@
     <inertial>
             <mass value="1.0"/>
-            <origin xyz="0 0 0"/>
             <inertia ixx="0.001458" iyy="0.001458" izz="0.00125" ixy="0.0" ixz="0.0" iyz="0.0"/>
     </inertial>
@@ -72,9 +70,9 @@
     <origin xyz="0.0 0.0 0.2" rpy="0.0 0.0 0.0"/>
     <parent link="base_link"/>
-    <child link="lidar"/>
+    <child link="lidar_link"/>
     <axis xyz="0.0 0.0 0.0"/>
     <limit lower="0.0" upper="0.0" effort="0.0" velocity="0.0"/>
 </joint>
-<gazebo reference="lidar">
+<gazebo reference="lidar_link">
     <sensor name="lidar" type="gpu_lidar">
       <ignition_frame_id>lidar_link</ignition_frame_id>
@@ -88,11 +86,11 @@
             <samples>360</samples>
             <resolution>1.000000</resolution>
-            <min_angle>0.000000</min_angle>
-            <max_angle>6.280000</max_angle>
+            <min_angle>-3.1400000</min_angle>
+            <max_angle>3.14</max_angle>
           </horizontal>
         </scan>
         <range>
-          <min>0.120000</min>
-          <max>3.5</max>
+          <min>0.3</min>
+          <max>12</max>
           <resolution>0.015000</resolution>
         </range>
@@ -103,4 +101,6 @@
         </noise>
       </ray>
+       <plugin filename="VisualizeLidar" name="Visualize Lidar">
+      </plugin>
     </sensor>
   </gazebo>

Commit message: new edit

File: description/4w_testbot.xacro (robot description, xacro)
@@ -50,5 +50,5 @@
 </joint>
 <!--Lidar properties-->
- <link name = "lidar_link">
+<link name = "lidar_link">
     <visual>
             <geometry>
@@ -71,11 +71,9 @@
     <parent link="base_link"/>
     <child link="lidar_link"/>
-    <axis xyz="0.0 0.0 0.0"/>
-    <limit lower="0.0" upper="0.0" effort="0.0" velocity="0.0"/>
 </joint>
 <gazebo reference="lidar_link">
     <sensor name="lidar" type="gpu_lidar">
       <ignition_frame_id>lidar_link</ignition_frame_id>
-      <topic>scan</topic>
+      <topic>lidar</topic>
       <always_on>true</always_on>
       <visualize>true</visualize>
@@ -101,6 +99,4 @@
         </noise>
       </ray>
-       <plugin filename="VisualizeLidar" name="Visualize Lidar">
-      </plugin>
     </sensor>
   </gazebo>

Commit message: added all edited files

File: description/4w_testbot.xacro (robot description, xacro)
@@ -20,13 +20,26 @@
   <xacro:macro name="box_inertia" params="m w h d">
     <inertial>
-      <origin xyz="0 0 0" rpy="${pi/2} 0 ${pi/2}"/>
+      <origin xyz="0 0 0.05" rpy="0 0 0"/>
       <mass value="${m}"/>
       <inertia ixx="${(m/12) * (h*h + d*d)}" ixy="0.0" ixz="0.0" iyy="${(m/12) * (w*w + d*d)}" iyz="0.0" izz="${(m/12) * (w*w + h*h)}"/>
     </inertial>
   </xacro:macro>
+  <xacro:macro name="cylinder_inertia" params="m r h">
+      <!--<origin xyz="0 0 ${0.3/2.0}" rpy="0 0 0"/>-->
+      <mass value="${m}"/>
+      <inertia  ixx="${m*(3*r*r+h*h)/12}" ixy = "0" ixz = "0"
+                  iyy="${m*(3*r*r+h*h)/12}" iyz = "0"
+                  izz="${m*r*r/2}" />
+      </xacro:macro>
 <!--- All Robots links with their full properties-->
-<!--Base_link properties-->
-<link name="base_footprint"/>
-<link name="base_link">
+<!--body_link properties-->
+<link name="base_footprint"> </link>
+<link name="base_link"> </link>
+<joint name = "base_body_footprint_joint" type = "fixed">
+<parent link="base_link"/>
+<child link = "body_link"/>
+<origin xyz="0.0 0.0 0.1" rpy="0.0 0.0 0.0" />
+</joint>
+<link name="body_link">
     <visual>
         <geometry>
@@ -42,10 +55,10 @@
         <origin xyz="0.0 0.0 0.05" rpy="0.0 0.0 0.0"/>
     </collision>
-    <xacro:box_inertia m="1.0" w="0.4" d="0.6" h="0.2"/>
+    <xacro:box_inertia m="2.5" w="0.4" d="0.6" h="0.2"/>
 </link>
 <joint name="base_link_footprint_joint" type="fixed">
-    <origin xyz="0.0 0.0 -0.15" rpy="0.0 0.0 0.0"/>
-    <parent link="base_link"/>
-    <child link="base_footprint"/>
+    <origin xyz="0.0 0.0 0" rpy="0.0 0.0 0.0"/>
+    <parent link="base_footprint"/>
+    <child link="base_link"/>
 </joint>
 <!--Lidar properties-->
@@ -63,4 +76,5 @@
     </collision>
     <inertial>
+            <origin xyz="0 0 0.2" rpy="0 0 0"/>
             <mass value="1.0"/>
             <inertia ixx="0.001458" iyy="0.001458" izz="0.00125" ixy="0.0" ixz="0.0" iyz="0.0"/>
@@ -68,10 +82,14 @@
 </link>
 <joint name="base_lidar" type="fixed">
-    <origin xyz="0.0 0.0 0.2" rpy="0.0 0.0 0.0"/>
-    <parent link="base_link"/>
+    <origin xyz="0.0 0.0 0.2" rpy="0.0 0.0 ${2*pi}"/>
+    <parent link="body_link"/>
     <child link="lidar_link"/>
 </joint>
+ <gazebo reference='base_lidar'>
+    <preserveFixedJoint>true</preserveFixedJoint>
+  </gazebo>
 <gazebo reference="lidar_link">
-    <sensor name="sensor_ray" type="gpu_lidar">
+    <sensor name="lidar" type="gpu_lidar">
+     <!-- <frame_id>lidar_link</frame_id>-->
       <ignition_frame_id>lidar_link</ignition_frame_id>
       <topic>/scan</topic>
@@ -89,6 +107,6 @@
         </scan>
         <range>
-          <min>0.3</min>
-          <max>12</max>
+          <min>0.03</min>
+          <max>10</max>
           <resolution>0.015000</resolution>
         </range>
@@ -125,5 +143,5 @@
 <joint name="${name}_joint" type="continuous">
     <origin xyz="${xyz}" rpy="0 0 0"/>
-    <parent link="base_link"/>
+    <parent link="body_link"/>
     <child link="${name}"/>
     <axis xyz="0.0 1.0 0.0"/>
@@ -132,7 +150,7 @@
 </xacro:macro>
 <!--definition of all four wheels-->
-<xacro:wheel name="rr_wheel" xyz="-0.18 -0.233 0.0" rpy="1.57 0 0" jrpy="3.142 0.0 0.0"/> <!--Rear right wheel-->
+<xacro:wheel name="rr_wheel" xyz="-0.18 -0.233 0.0" rpy="1.57 0 0" jrpy="0.0 0.0 0.0"/> <!--Rear right wheel-->
 <xacro:wheel name="fr_wheel" xyz="0.18 -0.233 0.0" rpy="1.57 0 0" jrpy="3.142 0.0 0.0"/><!--front right wheel-->
-<xacro:wheel name="fl_wheel" xyz="0.18 0.233 0.0" rpy="1.57 0 0" jrpy="0.0 0.0 0.0"/><!--front left wheel-->
+<xacro:wheel name="fl_wheel" xyz="0.18 0.233 0.0" rpy="1.57 0 0" jrpy="3.142 0.0 0.0"/><!--front left wheel-->
 <xacro:wheel name="rl_wheel" xyz="-0.18 0.233 0.0" rpy="1.57 0 0" jrpy="0.0 0.0 0.0"/><!--rear leftwheel-->
 <!---IMU properties-->
@@ -152,5 +170,5 @@
   </link>
    <joint name="imu_joint" type="fixed">
-    <parent link="base_link"/>
+    <parent link="body_link"/>
     <child link="imu_link"/>
     <origin xyz="0 0 0.01"/>
@@ -286,5 +304,5 @@
   </link>
   <joint name="camera_joint" type="fixed">
-    <parent link="base_link"/>
+    <parent link="body_link"/>
     <child link="camera_link"/>
     <origin xyz="0.309 0 0.1" rpy="0 0 0"/>

Commit message: Localizations and mapping

File: description/4w_testbot.xacro (robot description, xacro)
@@ -33,13 +33,13 @@
       </xacro:macro>
 <!--- All Robots links with their full properties-->
-<!--body_link properties-->
+<!--base_link properties-->
 <link name="base_footprint"> </link>
-<link name="base_link"> </link>
+<!--<link name="base_link"> </link>-->
 <joint name = "base_body_footprint_joint" type = "fixed">
-<parent link="base_link"/>
-<child link = "body_link"/>
+<parent link="base_footprint"/>
+<child link = "base_link"/>
 <origin xyz="0.0 0.0 0.1" rpy="0.0 0.0 0.0" />
 </joint>
-<link name="body_link">
+<link name="base_link">
     <visual>
         <geometry>
@@ -57,4 +57,5 @@
     <xacro:box_inertia m="2.5" w="0.4" d="0.6" h="0.2"/>
 </link>
+<!--
 <joint name="base_link_footprint_joint" type="fixed">
     <origin xyz="0.0 0.0 0" rpy="0.0 0.0 0.0"/>
@@ -62,4 +63,5 @@
     <child link="base_link"/>
 </joint>
+-->
 <!--Lidar properties-->
 <link name = "lidar_link">
@@ -83,5 +85,5 @@
 <joint name="base_lidar" type="fixed">
     <origin xyz="0.0 0.0 0.2" rpy="0.0 0.0 ${2*pi}"/>
-    <parent link="body_link"/>
+    <parent link="base_link"/>
     <child link="lidar_link"/>
 </joint>
@@ -105,4 +107,11 @@
             <max_angle>3.14</max_angle>
           </horizontal>
+          <!--use the vertical tag for 3D velodyne simulation-->
+         <!-- <vertical>
+          <resolution>1</resolution>
+              <samples>32</samples>
+              <min_angle>-0.5353</min_angle>
+              <max_angle>0.1862</max_angle>
+          </vertical> -->
         </scan>
         <range>
@@ -143,5 +152,5 @@
 <joint name="${name}_joint" type="continuous">
     <origin xyz="${xyz}" rpy="0 0 0"/>
-    <parent link="body_link"/>
+    <parent link="base_link"/>
     <child link="${name}"/>
     <axis xyz="0.0 1.0 0.0"/>
@@ -170,5 +179,5 @@
   </link>
    <joint name="imu_joint" type="fixed">
-    <parent link="body_link"/>
+    <parent link="base_link"/>
     <child link="imu_link"/>
     <origin xyz="0 0 0.01"/>
@@ -242,5 +251,5 @@
     <ros2_control name="IgnitionSystem" type="system">
     <hardware>
-      <plugin>ign_ros2_control/IgnitionSystem</plugin>
+      <plugin>gz_ros2_control/GazeboSimSystem</plugin>
     </hardware>
     <joint name="fr_wheel_joint">
@@ -278,5 +287,5 @@
   </ros2_control>
   <gazebo>
-    <plugin filename="ign_ros2_control-system" name="ign_ros2_control::IgnitionROS2ControlPlugin">
+    <plugin filename="gz_ros2_control-system" name="gz_ros2_control::GazeboSimROS2ControlPlugin">
       <parameters>$(find testbot)/config/4w_diff_drive_controller_velocity.yaml</parameters>
     </plugin>
@@ -304,7 +313,8 @@
   </link>
   <joint name="camera_joint" type="fixed">
-    <parent link="body_link"/>
+    <parent link="base_link"/>
     <child link="camera_link"/>
     <origin xyz="0.309 0 0.1" rpy="0 0 0"/>
+    <axis xyz='0 1 0'/>
   </joint>
   <link name="camera_frame"/>
@@ -315,5 +325,5 @@
   </joint>
   <gazebo reference="camera_link">
-    <sensor name="robot_cam" type="camera">
+    <sensor name="camera" type="camera">
       <camera>
         <horizontal_fov>1.047</horizontal_fov>
@@ -324,11 +334,18 @@
         <clip>
           <near>0.1</near>
-          <far>100</far>
+          <far>20</far>
         </clip>
+        <noise>
+          <type>gaussian</type>
+          <mean>0.0</mean>
+          <stddev>0.007</stddev>
+        </noise>
+        <optical_frame_id>camera_frame</optical_frame_id>
+        <camera_info_topic>camera_info</camera_info_topic>
       </camera>
       <always_on>1</always_on>
-      <update_rate>30</update_rate>
+      <update_rate>10</update_rate>
       <visualize>true</visualize>
-      <topic>robot_cam</topic>
+      <topic>/robot_cam</topic>
       <enable_metrics>true</enable_metrics>
     </sensor>
