Commit message: models and Nav2 Configs

File: description/4w_testbot.xacro (robot description, xacro)
@@ -1,21 +1,21 @@
 <?xml version="1.0"?>
-<robot xmlns:xacro="http://www.ros.org/wiki/xacro" name="roboct" >
-<!---materials definitions-->
-<material name="green">
+<robot xmlns:xacro="http://www.ros.org/wiki/xacro" name="roboct">
+  <!-- Materials -->
+  <material name="green">
     <color rgba="0.0 0.7 0.0 1.0"/>
-</material>
-<material name="blue">
-<color rgba="0.0 0.0 1.0 1.0"/>
-</material>
-<material name="red">
+  </material>
+  <material name="blue">
+    <color rgba="0.0 0.0 1.0 1.0"/>
+  </material>
+  <material name="red">
     <color rgba="1.0 0.0 0.0 1.0"/>
-</material>
-<material name="white">
+  </material>
+  <material name="white">
     <color rgba="1.0 1.0 1.0 1.0"/>
-</material>
-<material name="black">
+  </material>
+  <material name="black">
     <color rgba="0.0 0.0 0.0 1.0"/>
-</material>
-<!-- Define some commonly used intertial properties  -->
+  </material>
+  <!-- Inertia Macros -->
   <xacro:macro name="box_inertia" params="m w h d">
     <inertial>
@@ -26,72 +26,58 @@
   </xacro:macro>
   <xacro:macro name="cylinder_inertia" params="m r h">
-      <!--<origin xyz="0 0 ${0.3/2.0}" rpy="0 0 0"/>-->
+    <inertial>
       <mass value="${m}"/>
-      <inertia  ixx="${m*(3*r*r+h*h)/12}" ixy = "0" ixz = "0"
-                  iyy="${m*(3*r*r+h*h)/12}" iyz = "0"
-                  izz="${m*r*r/2}" />
-      </xacro:macro>
-<!--- All Robots links with their full properties-->
-<!--base_link properties-->
-<link name="base_footprint"> </link>
-<!--<link name="base_link"> </link>-->
-<joint name = "base_body_footprint_joint" type = "fixed">
-<parent link="base_footprint"/>
-<child link = "base_link"/>
-<origin xyz="0.0 0.0 0.1" rpy="0.0 0.0 0.0" />
-</joint>
-<link name="base_link">
+      <inertia ixx="${m*(3*r*r+h*h)/12}" ixy="0" ixz="0" iyy="${m*(3*r*r+h*h)/12}" iyz="0" izz="${m*r*r/2}"/>
+    </inertial>
+  </xacro:macro>
+  <!-- Base Footprint -->
+  <link name="base_footprint"></link>
+  <!-- Base Link -->
+  <link name="base_link">
     <visual>
-        <geometry>
-            <box size="0.6 0.4 0.2"/>
-        </geometry>
-        <origin xyz="0.0 0.0 0.05" rpy="0.0 0.0 0.0"/>
-        <material name="green"/>
+      <geometry>
+        <box size="0.6 0.4 0.2"/>
+      </geometry>
+      <origin xyz="0.0 0.0 0.05" rpy="0.0 0.0 0.0"/>
+      <material name="green"/>
     </visual>
     <collision>
-        <geometry>
-            <box size="0.6 0.4 0.2"/>
-        </geometry>
-        <origin xyz="0.0 0.0 0.05" rpy="0.0 0.0 0.0"/>
+      <geometry>
+        <box size="0.6 0.4 0.2"/>
+      </geometry>
+      <origin xyz="0.0 0.0 0.05" rpy="0.0 0.0 0.0"/>
     </collision>
     <xacro:box_inertia m="2.5" w="0.4" d="0.6" h="0.2"/>
-</link>
-<!--
-<joint name="base_link_footprint_joint" type="fixed">
-    <origin xyz="0.0 0.0 0" rpy="0.0 0.0 0.0"/>
+  </link>
+  <joint name="base_body_footprint_joint" type="fixed">
     <parent link="base_footprint"/>
     <child link="base_link"/>
-</joint>
--->
-<!--Lidar properties-->
-<link name = "lidar_link">
+    <origin xyz="0.0 0.0 0.1" rpy="0.0 0.0 0.0"/>
+  </joint>
+  <!-- LIDAR -->
+  <link name="lidar_link">
     <visual>
-            <geometry>
-                <cylinder radius="0.0808" length="0.055"/>
-            </geometry>
-            <material name="black"/>
+      <geometry>
+        <cylinder radius="0.0808" length="0.055"/>
+      </geometry>
+      <material name="black"/>
     </visual>
     <collision>
-        <geometry>
-            <cylinder radius="0.0808" length="0.055"/>
-        </geometry>
+      <geometry>
+        <cylinder radius="0.0808" length="0.055"/>
+      </geometry>
     </collision>
-    <inertial>
-            <origin xyz="0 0 0.2" rpy="0 0 0"/>
-            <mass value="1.0"/>
-            <inertia ixx="0.001458" iyy="0.001458" izz="0.00125" ixy="0.0" ixz="0.0" iyz="0.0"/>
-    </inertial>
-</link>
-<joint name="base_lidar" type="fixed">
-    <origin xyz="0.0 0.0 0.2" rpy="0.0 0.0 ${2*pi}"/>
+    <xacro:cylinder_inertia m="1.0" r="0.0808" h="0.055"/>
+  </link>
+  <joint name="base_lidar" type="fixed">
+    <origin xyz="0.0 0.0 0.2" rpy="0 0 0"/>
     <parent link="base_link"/>
     <child link="lidar_link"/>
-</joint>
- <gazebo reference='base_lidar'>
+  </joint>
+  <gazebo reference="base_lidar">
     <preserveFixedJoint>true</preserveFixedJoint>
   </gazebo>
-<gazebo reference="lidar_link">
+  <gazebo reference="lidar_link">
     <sensor name="lidar" type="gpu_lidar">
-     <!-- <frame_id>lidar_link</frame_id>-->
       <ignition_frame_id>lidar_link</ignition_frame_id>
       <topic>/scan</topic>
@@ -103,20 +89,13 @@
           <horizontal>
             <samples>360</samples>
-            <resolution>1.000000</resolution>
-            <min_angle>-3.1400000</min_angle>
+            <resolution>1.0</resolution>
+            <min_angle>-3.14</min_angle>
             <max_angle>3.14</max_angle>
           </horizontal>
-          <!--use the vertical tag for 3D velodyne simulation-->
-         <!-- <vertical>
-          <resolution>1</resolution>
-              <samples>32</samples>
-              <min_angle>-0.5353</min_angle>
-              <max_angle>0.1862</max_angle>
-          </vertical> -->
         </scan>
         <range>
           <min>0.03</min>
           <max>10</max>
-          <resolution>0.015000</resolution>
+          <resolution>0.015</resolution>
         </range>
         <noise>
@@ -128,64 +107,53 @@
     </sensor>
   </gazebo>
-<!--Wheel properties-->
-<xacro:macro name="wheel" params="name xyz rpy jrpy">
-<link name = "${name}">
-    <visual>
-            <geometry>
-                <cylinder radius="0.1" length="0.05"/>
-            </geometry>
-            <origin xyz="0.0 0.0 0.0" rpy="${rpy}"/>
-            <material name="blue"/>
-    </visual>
-    <collision>
+  <!-- Wheels -->
+  <xacro:macro name="wheel" params="name xyz rpy">
+    <link name="${name}">
+      <visual>
         <geometry>
-            <cylinder radius="0.1" length="0.05"/>
+          <cylinder radius="0.1" length="0.05"/>
         </geometry>
         <origin xyz="0.0 0.0 0.0" rpy="${rpy}"/>
-    </collision>
-    <inertial>
-            <mass value="1.0"/>
-            <origin xyz="0 0 0"/>
-            <inertia ixx="0.001458" iyy="0.001458" izz="0.00125" ixy="0.0" ixz="0.0" iyz="0.0"/>
-    </inertial>
-</link>
-<joint name="${name}_joint" type="continuous">
-    <origin xyz="${xyz}" rpy="0 0 0"/>
-    <parent link="base_link"/>
-    <child link="${name}"/>
-    <axis xyz="0.0 1.0 0.0"/>
-    <dynamics damping="0.2"/>
-</joint>
-</xacro:macro>
-<!--definition of all four wheels-->
-<xacro:wheel name="rr_wheel" xyz="-0.18 -0.233 0.0" rpy="1.57 0 0" jrpy="0.0 0.0 0.0"/> <!--Rear right wheel-->
-<xacro:wheel name="fr_wheel" xyz="0.18 -0.233 0.0" rpy="1.57 0 0" jrpy="3.142 0.0 0.0"/><!--front right wheel-->
-<xacro:wheel name="fl_wheel" xyz="0.18 0.233 0.0" rpy="1.57 0 0" jrpy="3.142 0.0 0.0"/><!--front left wheel-->
-<xacro:wheel name="rl_wheel" xyz="-0.18 0.233 0.0" rpy="1.57 0 0" jrpy="0.0 0.0 0.0"/><!--rear leftwheel-->
-<!---IMU properties-->
-<link name="imu_link">
-    <visual>
-      <geometry>
-        <box size="0.1 0.1 0.1"/>
-      </geometry>
-      <material name="red"/>
-    </visual>
-    <collision>
-      <geometry>
-        <box size="0.1 0.1 0.1"/>
-      </geometry>
-    </collision>
-    <xacro:box_inertia m="0.001" w="0.1" d="0.1" h="0.1"/>
-  </link>
-   <joint name="imu_joint" type="fixed">
+        <material name="blue"/>
+      </visual>
+      <collision>
+        <geometry>
+          <cylinder radius="0.1" length="0.05"/>
+        </geometry>
+        <origin xyz="0.0 0.0 0.0" rpy="${rpy}"/>
+        <surface>
+          <friction>
+            <ode>
+              <mu>1.0</mu>
+              <mu2>1.0</mu2>
+            </ode>
+          </friction>
+        </surface>
+      </collision>
+      <xacro:cylinder_inertia m="1.0" r="0.1" h="0.05"/>
+    </link>
+    <joint name="${name}_joint" type="continuous">
+      <origin xyz="${xyz}" rpy="0 0 0"/>
+      <parent link="base_link"/>
+      <child link="${name}"/>
+      <axis xyz="0.0 1.0 0.0"/>
+      <dynamics damping="0.2"/>
+    </joint>
+  </xacro:macro>
+  <xacro:wheel name="rr_wheel" xyz="-0.18 -0.233 0.0" rpy="1.57 0 0"/>
+  <xacro:wheel name="fr_wheel" xyz="0.18 -0.233 0.0" rpy="1.57 0 0"/>
+  <xacro:wheel name="fl_wheel" xyz="0.18 0.233 0.0" rpy="1.57 0 0"/>
+  <xacro:wheel name="rl_wheel" xyz="-0.18 0.233 0.0" rpy="1.57 0 0"/>
+  <!-- IMU -->
+  <link name="imu_link"/>
+  <joint name="imu_joint" type="fixed">
     <parent link="base_link"/>
     <child link="imu_link"/>
-    <origin xyz="0 0 0.01"/>
+    <origin xyz="0 0 0.01" rpy="0 0 0"/>
   </joint>
   <gazebo reference="imu_link">
     <sensor name="imu_sensor" type="imu">
       <ignition_frame_id>imu_link</ignition_frame_id>
-      <plugin filename="ignition-gazebo-imu-system" name="ignition::gazebo::systems::Imu">
-      </plugin>
+      <plugin filename="ignition-gazebo-imu-system" name="ignition::gazebo::systems::Imu"/>
       <topic>imu</topic>
       <always_on>true</always_on>
@@ -248,6 +216,6 @@
     </sensor>
   </gazebo>
-    <!--Control ad gazebo control interface-->
-    <ros2_control name="IgnitionSystem" type="system">
+  <!-- ROS2 Control -->
+  <ros2_control name="IgnitionSystem" type="system">
     <hardware>
       <plugin>gz_ros2_control/GazeboSimSystem</plugin>
@@ -255,6 +223,6 @@
     <joint name="fr_wheel_joint">
       <command_interface name="velocity">
-        <param name="min">-1</param>
-        <param name="max">1</param>
+        <param name="min">-5</param>
+        <param name="max">5</param>
       </command_interface>
       <state_interface name="position"/>
@@ -263,6 +231,6 @@
     <joint name="rr_wheel_joint">
       <command_interface name="velocity">
-        <param name="min">-1</param>
-        <param name="max">1</param>
+        <param name="min">-5</param>
+        <param name="max">5</param>
       </command_interface>
       <state_interface name="position"/>
@@ -271,6 +239,6 @@
     <joint name="fl_wheel_joint">
       <command_interface name="velocity">
-        <param name="min">-1</param>
-        <param name="max">1</param>
+        <param name="min">-5</param>
+        <param name="max">5</param>
       </command_interface>
       <state_interface name="position"/>
@@ -279,6 +247,6 @@
     <joint name="rl_wheel_joint">
       <command_interface name="velocity">
-        <param name="min">-1</param>
-        <param name="max">1</param>
+        <param name="min">-5</param>
+        <param name="max">5</param>
       </command_interface>
       <state_interface name="position"/>
@@ -291,5 +259,5 @@
     </plugin>
   </gazebo>
-  <!--Camera properties-->
+  <!-- Camera -->
   <link name="camera_link">
     <visual>
@@ -307,7 +275,6 @@
     </collision>
     <inertial>
-      <origin xyz="0 0 0" rpy="0 0 0"/>
       <mass value="0.035"/>
-      <inertia ixx="0.001" ixy="0" ixz="0" iyy="0.001" iyz="0" izz="0.001" />
+      <inertia ixx="1.8e-6" iyy="4.9e-5" izz="5.0e-5" ixy="0" ixz="0" iyz="0"/>
     </inertial>
   </link>
@@ -316,5 +283,5 @@
     <child link="camera_link"/>
     <origin xyz="0.309 0 0.1" rpy="0 0 0"/>
-    <axis xyz='0 1 0'/>
+    <axis xyz="0 1 0"/>
   </joint>
   <link name="camera_frame"/>
